Commit message: add lidar pkg

File: src/mybot_pkg/urdf/LibraryBot.urdf (robot description, URDF)
Before this commit: robot LibraryBot, 7 links, 6 joints
Links:
- removed link base_footprint
Joints:
- removed joint joint base

Commit message: update navigation parameters

File: src/mybot_pkg/urdf/LibraryBot.urdf (robot description, URDF)
Before this commit: robot LibraryBot, 6 links, 5 joints
Joints:
- joint lidar_joint: origin xyz=0 0 0.1025 rpy=0 0 0 -> xyz=0 0 0.0 rpy=0 0 0
