Commit message: final commit before presentation

File: src/mybot_pkg/urdf/LibraryBot_simulation.urdf (robot description, URDF)
Before this commit: robot LibraryBot, 6 links, 5 joints
Links:
- removed link lidar_link
- added link laser, mass 1.0; collision cylinder length=0.023 radius=0.039; visual cylinder length=0.023 radius=0.039
Joints:
- joint lidar_joint: child lidar_link -> laser
